File: tinybee_v1.sch (EAGLE design)
At the start: 21 parts, among them U1 ATTINY85-20S

Commit message: route
Parts:
- removed FRAME1: FRAME-LETTER, SparkFun-Aesthetics:FRAME-LETTER
Changed lines of the file:
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@@
 <?xml version="1.0" encoding="utf-8"?>
 <!DOCTYPE eagle SYSTEM "eagle.dtd">
-<eagle version="7.3.0">
+<eagle version="7.2.0">
 <drawing>
 <settings>
@@
 </classes>
 <parts>
-<part name="FRAME1" library="SparkFun-Aesthetics" deviceset="FRAME-LETTER" device=""/>
 <part name="U1" library="_hhn_attiny25_45_85" deviceset="ATTINY85*" device="S" technology="-20"/>
 <part name="GND1" library="SparkFun-Aesthetics" deviceset="GND" device=""/>
@@
 </plain>
 <instances>
-<instance part="FRAME1" gate="G$1" x="0" y="0"/>
-<instance part="FRAME1" gate="V" x="147.32" y="0"/>
 <instance part="U1" gate="G$1" x="50.8" y="114.3"/>
 <instance part="GND1" gate="1" x="101.6" y="86.36"/>
