File: tinybee_v1.sch (EAGLE design)
At the start: 21 parts, among them U1 ATTINY85-20S

Commit message: Fixes after Eran review
Connections:
- net N$1 renamed VBUS
- removed net N$5: C1.1, U1.VCC
- net GND: now also C1.2
- net VCC: now also C1.1, U1.VCC; no longer C1.2
Other:
- moved on the sheet: C1
Changed lines of the file:
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@@
 <instance part="GND3" gate="1" x="30.48" y="99.06"/>
 <instance part="SUPPLY1" gate="G$1" x="139.7" y="76.2"/>
-<instance part="SUPPLY2" gate="G$1" x="20.32" y="127"/>
+<instance part="SUPPLY2" gate="G$1" x="30.48" y="121.92"/>
 <instance part="USB" gate="G$1" x="137.16" y="116.84" rot="R180"/>
 <instance part="SUPPLY3" gate="G$1" x="101.6" y="137.16"/>
@@
 <instance part="SUPPLY4" gate="G$1" x="190.5" y="132.08"/>
 <instance part="GND5" gate="1" x="162.56" y="96.52"/>
-<instance part="C1" gate="G$1" x="25.4" y="119.38" rot="R270"/>
+<instance part="C1" gate="G$1" x="30.48" y="111.76"/>
 <instance part="C2" gate="G$1" x="114.3" y="93.98"/>
 <instance part="GND6" gate="1" x="114.3" y="86.36"/>
@@
 </segment>
 <segment>
-<pinref part="SUPPLY2" gate="G$1" pin="VCC"/>
-<wire x1="20.32" y1="127" x2="20.32" y2="119.38" width="0.1524" layer="91"/>
-<pinref part="C1" gate="G$1" pin="2"/>
-<wire x1="20.32" y1="119.38" x2="22.86" y2="119.38" width="0.1524" layer="91"/>
-</segment>
-<segment>
 <pinref part="R8" gate="G$1" pin="2"/>
 <pinref part="SUPPLY4" gate="G$1" pin="VCC"/>
@@
 <junction x="114.3" y="106.68"/>
 </segment>
+<segment>
+<pinref part="C1" gate="G$1" pin="1"/>
+<pinref part="SUPPLY2" gate="G$1" pin="VCC"/>
+<wire x1="30.48" y1="116.84" x2="30.48" y2="119.38" width="0.1524" layer="91"/>
+<pinref part="U1" gate="G$1" pin="VCC"/>
+<wire x1="30.48" y1="119.38" x2="30.48" y2="121.92" width="0.1524" layer="91"/>
+<wire x1="35.56" y1="119.38" x2="30.48" y2="119.38" width="0.1524" layer="91"/>
+<junction x="30.48" y="119.38"/>
+</segment>
 </net>
 <net name="GND" class="0">
@@
 <pinref part="GND3" gate="1" pin="GND"/>
 <wire x1="30.48" y1="106.68" x2="30.48" y2="101.6" width="0.1524" layer="91"/>
+<pinref part="C1" gate="G$1" pin="2"/>
+<wire x1="30.48" y1="109.22" x2="30.48" y2="106.68" width="0.1524" layer="91"/>
+<junction x="30.48" y="106.68"/>
 </segment>
 <segment>
@@
 </segment>
 </net>
-<net name="N$5" class="0">
-<segment>
-<pinref part="C1" gate="G$1" pin="1"/>
-<pinref part="U1" gate="G$1" pin="VCC"/>
-<wire x1="30.48" y1="119.38" x2="35.56" y2="119.38" width="0.1524" layer="91"/>
-</segment>
-</net>
 <net name="PB4" class="0">
 <segment>
@@
 <wire x1="81.28" y1="116.84" x2="68.58" y2="116.84" width="0.1524" layer="91"/>
 <pinref part="R3" gate="G$1" pin="1"/>
+<label x="68.58" y="116.84" size="1.778" layer="95"/>
 </segment>
 </net>
@@
 <wire x1="73.66" y1="114.3" x2="68.58" y2="114.3" width="0.1524" layer="91"/>
 <pinref part="R2" gate="G$1" pin="1"/>
+<label x="68.58" y="114.3" size="1.778" layer="95"/>
 </segment>
 <segment>
@@
 <pinref part="U1" gate="G$1" pin="PB2"/>
 <wire x1="68.58" y1="111.76" x2="73.66" y2="111.76" width="0.1524" layer="91"/>
+<label x="68.58" y="111.76" size="1.778" layer="95"/>
 </segment>
 <segment>
@@
 <pinref part="U1" gate="G$1" pin="PB1"/>
 <wire x1="68.58" y1="109.22" x2="73.66" y2="109.22" width="0.1524" layer="91"/>
+<label x="68.58" y="109.22" size="1.778" layer="95"/>
 </segment>
 <segment>
@@
 <pinref part="U1" gate="G$1" pin="PB0"/>
 <wire x1="68.58" y1="106.68" x2="73.66" y2="106.68" width="0.1524" layer="91"/>
+<label x="68.58" y="106.68" size="1.778" layer="95"/>
 </segment>
 <segment>
@@
 <pinref part="U1" gate="G$1" pin="NRES/PB5"/>
 <wire x1="68.58" y1="119.38" x2="73.66" y2="119.38" width="0.1524" layer="91"/>
+<label x="68.58" y="119.38" size="1.778" layer="95"/>
 </segment>
 <segment>
@@
 </segment>
 </net>
-<net name="N$1" class="0">
+<net name="VBUS" class="0">
 <segment>
 <pinref part="USB" gate="G$1" pin="VBUS"/>
 <pinref part="S1" gate="G$1" pin="1"/>
 <wire x1="127" y1="111.76" x2="121.92" y2="111.76" width="0.1524" layer="91"/>
-</segment>
-</net>
+<label x="121.92" y="111.76" size="1.778" layer="95"/>
+</segment>
+</net>

Commit message: routing
Parts:
- C1: device SparkFun-Capacitors:0.1UF-25V(+80/-20%)(0603) -> microbuilder:CAP_CERAMIC0603
Connections:
- net GND: now also C1.P$1; no longer C1.2
- net PB0: now also R4.1; no longer C3.P$2, R6.2
- net PB1: now also C3.P$2, R6.2; no longer C4.P$2, R5.2
- net PB2: now also C4.P$2, R5.2; no longer R4.1
- net VCC: now also C1.P$2; no longer C1.1
Other:
- moved on the sheet: C1
Changed lines of the file:
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@@
 <part name="SUPPLY4" library="SparkFun-Aesthetics" deviceset="VCC" device=""/>
 <part name="GND5" library="SparkFun-Aesthetics" deviceset="GND" device=""/>
-<part name="C1" library="SparkFun-Capacitors" deviceset="0.1UF-25V(+80/-20%)(0603)" device="" value="0.1uF"/>
 <part name="C2" library="microbuilder" deviceset="CAP_ELECTROLYTIC" device="PANASONIC_C" value="47uF"/>
 <part name="GND6" library="SparkFun-Aesthetics" deviceset="GND" device=""/>
@@
 <part name="GND9" library="SparkFun-Aesthetics" deviceset="GND" device=""/>
 <part name="S1" library="Custom" deviceset="SWITCH-SLIDE-SPDT-RIGHTANGLE-500" device=""/>
+<part name="C1" library="microbuilder" deviceset="CAP_CERAMIC" device="0603" value="0.1uF"/>
 </parts>
 <sheets>
@@
 <instance part="SUPPLY4" gate="G$1" x="190.5" y="132.08"/>
 <instance part="GND5" gate="1" x="162.56" y="96.52"/>
-<instance part="C1" gate="G$1" x="30.48" y="111.76"/>
 <instance part="C2" gate="G$1" x="114.3" y="93.98"/>
 <instance part="GND6" gate="1" x="114.3" y="86.36"/>
@@
 <instance part="GND9" gate="1" x="193.04" y="96.52"/>
 <instance part="S1" gate="G$1" x="119.38" y="109.22"/>
+<instance part="C1" gate="G$1" x="30.48" y="114.3" rot="R180"/>
 </instances>
 <busses>
@@
 </segment>
 <segment>
-<pinref part="C1" gate="G$1" pin="1"/>
 <pinref part="SUPPLY2" gate="G$1" pin="VCC"/>
 <wire x1="30.48" y1="116.84" x2="30.48" y2="119.38" width="0.1524" layer="91"/>
@@
 <wire x1="35.56" y1="119.38" x2="30.48" y2="119.38" width="0.1524" layer="91"/>
 <junction x="30.48" y="119.38"/>
+<pinref part="C1" gate="G$1" pin="P$2"/>
 </segment>
 </net>
@@
 <pinref part="GND3" gate="1" pin="GND"/>
 <wire x1="30.48" y1="106.68" x2="30.48" y2="101.6" width="0.1524" layer="91"/>
-<pinref part="C1" gate="G$1" pin="2"/>
 <wire x1="30.48" y1="109.22" x2="30.48" y2="106.68" width="0.1524" layer="91"/>
 <junction x="30.48" y="106.68"/>
+<pinref part="C1" gate="G$1" pin="P$1"/>
 </segment>
 <segment>
@@
 </segment>
 <segment>
-<wire x1="132.08" y1="71.12" x2="124.46" y2="71.12" width="0.1524" layer="91"/>
-<label x="121.92" y="71.12" size="1.778" layer="95"/>
-<pinref part="R4" gate="G$1" pin="1"/>
-</segment>
-<segment>
 <pinref part="JP2" gate="G$1" pin="3"/>
 <wire x1="40.64" y1="71.12" x2="38.1" y2="71.12" width="0.1524" layer="91"/>
 <label x="30.48" y="71.12" size="1.778" layer="95"/>
-</segment>
-</net>
-<net name="PB1" class="0">
-<segment>
-<pinref part="U1" gate="G$1" pin="PB1"/>
-<wire x1="68.58" y1="109.22" x2="73.66" y2="109.22" width="0.1524" layer="91"/>
-<label x="68.58" y="109.22" size="1.778" layer="95"/>
 </segment>
 <segment>
@@
 <junction x="220.98" y="114.3"/>
 </segment>
+</net>
+<net name="PB1" class="0">
+<segment>
+<pinref part="U1" gate="G$1" pin="PB1"/>
+<wire x1="68.58" y1="109.22" x2="73.66" y2="109.22" width="0.1524" layer="91"/>
+<label x="68.58" y="109.22" size="1.778" layer="95"/>
+</segment>
 <segment>
 <pinref part="JP2" gate="G$1" pin="1"/>
 <wire x1="40.64" y1="73.66" x2="38.1" y2="73.66" width="0.1524" layer="91"/>
 <label x="30.48" y="73.66" size="1.778" layer="95"/>
-</segment>
-</net>
-<net name="PB0" class="0">
-<segment>
-<pinref part="U1" gate="G$1" pin="PB0"/>
-<wire x1="68.58" y1="106.68" x2="73.66" y2="106.68" width="0.1524" layer="91"/>
-<label x="68.58" y="106.68" size="1.778" layer="95"/>
 </segment>
 <segment>
@@
 <junction x="210.82" y="104.14"/>
 </segment>
+</net>
+<net name="PB0" class="0">
+<segment>
+<pinref part="U1" gate="G$1" pin="PB0"/>
+<wire x1="68.58" y1="106.68" x2="73.66" y2="106.68" width="0.1524" layer="91"/>
+<label x="68.58" y="106.68" size="1.778" layer="95"/>
+</segment>
 <segment>
 <pinref part="JP2" gate="G$1" pin="4"/>
@@
 <label x="62.23" y="71.12" size="1.778" layer="95"/>
 </segment>
-</net>
+<segment>
+<wire x1="132.08" y1="71.12" x2="124.46" y2="71.12" width="0.1524" layer="91"/>
+<label x="121.92" y="71.12" size="1.778" layer="95"/>
+<pinref part="R4" gate="G$1" pin="1"/>
+</segment>
+</net>
