File: tinybee_v1.brd (EAGLE design)
At the start: 47.6 x 27.8 mm, 22 parts, among them U1 ATTINY85-20S

Commit message: Final touches. Redid USB connector footprint
Parts:
- moved USB 0.25 mm to (4.06, 8.51)
- moved R1 0.13 mm to (7.49, 10.4)
Routing:
- net VBUS: track 13.8 -> 16.4 mm
- net VCC: track 16.3 -> 18.1 mm
Other:
- board text added: "TinyBee v1"
